File: v1/SwitchMatrixPCB/schematics.kicad_sch (KiCad schematic)
At the start: 175 parts, among them U1 ESP32-S3-DevKitC

Commit message: New Schematic files (v2_TEMP)
Parts:
- removed U1: ESP32-S3-DevKitC, PCM_Espressif:ESP32-S3-DevKitC, symbol PCM_Espressif:ESP32-S3-DevKitC
- added D88: Diode, ScottoKeebs_Components:Diode_DO-35, symbol ScottoKeebs:Placeholder_Diode
- added S88: Keyswitch, ScottoKeebs_MX:MX_PCB_1.00u, symbol ScottoKeebs:Placeholder_Keyswitch
Connections:
- net Col 01: now also S88.1
- net Row 3: now also D88.1 (K)
- new net: D88.2 (A), S88.2
Other:
- moved on the sheet: D6, S6
