File: v2/Matrix/v2.kicad_pcb (KiCad board)
At the start: 2 copper layers, 366 parts, among them J2 Conn_01x16, K0 ESC, K1 F1, K10 F10, K11 F11, K12 F12, K13 <i class='kb kb-Unicode-Print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, K14 INS, K15 DEL, K16 |,\, K17 !,,,,,,,,,1, K18 ",@,,,,,,,,2, K19 #,£,,,,,,,,3, K2 F2, K20 $,§,,,,,,,,4, K21 %,€,,,,,,,,5, K22 &,,,,,,,,,6, K23 /,{,,,,,,,,7, K24 (,[,,,,,,,,8, K25 ),],,,,,,,,9, K26 =,},,,,,,,,0, K27 ?,', K28 »,«, K29 BACKSPACE, K3 F3, K30 Blank, K31 PGUP, K32 TAB, K33 Q, K34 W, K35 E, K36 R, K37 T, K38 Y, K39 U, K4 F4, K40 I, K41 O, K42 P, K43 *,+, K44 `,´, K45 |,\, K46 PGDN, K47 CAPS, K48 A, K49 S, K5 F5, K50 D, K51 F, K52 G, K53 H, K54 J, K55 K, K56 L, K57 Ç, K58 ª,º, K59 ^,~, K59 ^,~~, K6 F6, K60 ENTER, K61 HOME, K62 SHIFT, K63 Z, K64 X, K65 C, K66 V, K67 B, K68 N, K69 M, K7 F7, K70 ;,,, K71 :,., K72 -,_, K73 >,,,,,,,,,<, K74 SHIFT, K75 END, K76 ∧, K77 Blank, K78 CTRL, K79 SUPER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

Commit message: Updated the kicad schematics.
Parts:
- added D100: Diode, ScottoKeebs_Components:Diode_SOD-123, F.Cu at (426.3, 97.5)
- added D101: Diode, ScottoKeebs_Components:Diode_SOD-123, F.Cu at (426.3, 101.1)
- added D102: Diode, ScottoKeebs_Components:Diode_SOD-123, F.Cu at (426.3, 104.7)
- added D103: Diode, ScottoKeebs_Components:Diode_SOD-123, F.Cu at (426.3, 108.2)
- added D104: Diode, ScottoKeebs_Components:Diode_SOD-123, F.Cu at (426.3, 111.8)
- added D105: Diode, ScottoKeebs_Components:Diode_SOD-123, F.Cu at (426.3, 115.3)
- added D106: Diode, ScottoKeebs_Components:Diode_SOD-123, F.Cu at (426.3, 118.8)
- added D107: Diode, ScottoKeebs_Components:Diode_SOD-123, F.Cu at (426.3, 122.4)
- added D108: Diode, ScottoKeebs_Components:Diode_SOD-123, F.Cu at (437.0, 62.0)
- added D109: Diode, ScottoKeebs_Components:Diode_SOD-123, F.Cu at (437.0, 65.6)
- added D110: Diode, ScottoKeebs_Components:Diode_SOD-123, F.Cu at (437.0, 69.2)
- added D111: Diode, ScottoKeebs_Components:Diode_SOD-123, F.Cu at (437.0, 72.7)
- added D112: Diode, ScottoKeebs_Components:Diode_SOD-123, F.Cu at (437.0, 76.2)
- added D113: Diode, ScottoKeebs_Components:Diode_SOD-123, F.Cu at (437.0, 79.8)
- added D114: Diode, ScottoKeebs_Components:Diode_SOD-123, F.Cu at (437.0, 83.3)
- added D115: Diode, ScottoKeebs_Components:Diode_SOD-123, F.Cu at (437.0, 86.9)
- added D116: Diode, ScottoKeebs_Components:Diode_SOD-123, F.Cu at (437.0, 90.5)
- added D117: Diode, ScottoKeebs_Components:Diode_SOD-123, F.Cu at (437.0, 94.0)
- added D118: Diode, ScottoKeebs_Components:Diode_SOD-123, F.Cu at (437.0, 97.5)
- added D119: Diode, ScottoKeebs_Components:Diode_SOD-123, F.Cu at (437.0, 101.1)
- added D120: Diode, ScottoKeebs_Components:Diode_SOD-123, F.Cu at (437.0, 104.7)
- added D121: Diode, ScottoKeebs_Components:Diode_SOD-123, F.Cu at (437.0, 108.2)
- added D122: Diode, ScottoKeebs_Components:Diode_SOD-123, F.Cu at (437.0, 111.8)
- added D123: Diode, ScottoKeebs_Components:Diode_SOD-123, F.Cu at (437.0, 115.3)
- added D124: Diode, ScottoKeebs_Components:Diode_SOD-123, F.Cu at (437.0, 118.8)
- added D125: Diode, ScottoKeebs_Components:Diode_SOD-123, F.Cu at (437.0, 122.4)
- added D126: Diode, ScottoKeebs_Components:Diode_SOD-123, F.Cu at (447.8, 62.0)
- added D127: Diode, ScottoKeebs_Components:Diode_SOD-123, F.Cu at (447.8, 65.6)
- added D128: Diode, ScottoKeebs_Components:Diode_SOD-123, F.Cu at (447.8, 69.2)
- added D129: Diode, ScottoKeebs_Components:Diode_SOD-123, F.Cu at (447.8, 72.7)
- added D130: Diode, ScottoKeebs_Components:Diode_SOD-123, F.Cu at (447.8, 76.2)
- added D131: Diode, ScottoKeebs_Components:Diode_SOD-123, F.Cu at (447.8, 79.8)
- added D132: Diode, ScottoKeebs_Components:Diode_SOD-123, F.Cu at (447.8, 83.3)
- added D133: Diode, ScottoKeebs_Components:Diode_SOD-123, F.Cu at (447.8, 86.9)
- added D134: Diode, ScottoKeebs_Components:Diode_SOD-123, F.Cu at (447.8, 90.5)
- added D135: Diode, ScottoKeebs_Components:Diode_SOD-123, F.Cu at (447.8, 94.0)
- added D136: Diode, ScottoKeebs_Components:Diode_SOD-123, F.Cu at (447.8, 97.5)
- added D137: Diode, ScottoKeebs_Components:Diode_SOD-123, F.Cu at (447.8, 101.1)
- added D138: Diode, ScottoKeebs_Components:Diode_SOD-123, F.Cu at (447.8, 104.7)
- added D139: Diode, ScottoKeebs_Components:Diode_SOD-123, F.Cu at (447.8, 108.2)
- added D140: Diode, ScottoKeebs_Components:Diode_SOD-123, F.Cu at (447.8, 111.8)
- added D141: Diode, ScottoKeebs_Components:Diode_SOD-123, F.Cu at (447.8, 115.3)
- added D142: Diode, ScottoKeebs_Components:Diode_SOD-123, F.Cu at (447.8, 118.8)
- added D143: Diode, ScottoKeebs_Components:Diode_SOD-123, F.Cu at (447.8, 122.4)
- added D144: Diode, ScottoKeebs_Components:Diode_SOD-123, F.Cu at (458.6, 62.0)
- added D145: Diode, ScottoKeebs_Components:Diode_SOD-123, F.Cu at (458.6, 65.6)
- added D146: Diode, ScottoKeebs_Components:Diode_SOD-123, F.Cu at (458.6, 69.2)
- added D147: Diode, ScottoKeebs_Components:Diode_SOD-123, F.Cu at (458.6, 72.7)
- added D148: Diode, ScottoKeebs_Components:Diode_SOD-123, F.Cu at (458.6, 76.2)
- added D149: Diode, ScottoKeebs_Components:Diode_SOD-123, F.Cu at (458.6, 79.8)
- added D150: Diode, ScottoKeebs_Components:Diode_SOD-123, F.Cu at (458.6, 83.3)
- added D151: Diode, ScottoKeebs_Components:Diode_SOD-123, F.Cu at (458.6, 86.9)
- added D152: Diode, ScottoKeebs_Components:Diode_SOD-123, F.Cu at (458.6, 90.5)
- added D153: Diode, ScottoKeebs_Components:Diode_SOD-123, F.Cu at (458.6, 94.0)
- added D154: Diode, ScottoKeebs_Components:Diode_SOD-123, F.Cu at (458.6, 97.5)
- added D155: Diode, ScottoKeebs_Components:Diode_SOD-123, F.Cu at (458.6, 101.1)
- added D156: Diode, ScottoKeebs_Components:Diode_SOD-123, F.Cu at (458.6, 104.7)
- added D157: Diode, ScottoKeebs_Components:Diode_SOD-123, F.Cu at (458.6, 108.2)
- added D158: Diode, ScottoKeebs_Components:Diode_SOD-123, F.Cu at (458.6, 111.8)
- added D159: Diode, ScottoKeebs_Components:Diode_SOD-123, F.Cu at (458.6, 115.3)
- added D160: Diode, ScottoKeebs_Components:Diode_SOD-123, F.Cu at (458.6, 118.8)
- added D161: Diode, ScottoKeebs_Components:Diode_SOD-123, F.Cu at (458.6, 122.4)
- added D162: Diode, ScottoKeebs_Components:Diode_SOD-123, F.Cu at (469.4, 62.0)
- added D163: Diode, ScottoKeebs_Components:Diode_SOD-123, F.Cu at (469.4, 65.6)
- added D164: Diode, ScottoKeebs_Components:Diode_SOD-123, F.Cu at (469.4, 69.2)
- added D165: Diode, ScottoKeebs_Components:Diode_SOD-123, F.Cu at (469.4, 72.7)
- added D166: Diode, ScottoKeebs_Components:Diode_SOD-123, F.Cu at (469.4, 76.2)
- added D167: Diode, ScottoKeebs_Components:Diode_SOD-123, F.Cu at (469.4, 79.8)
- added D168: Diode, ScottoKeebs_Components:Diode_SOD-123, F.Cu at (469.4, 83.3)
- added D169: Diode, ScottoKeebs_Components:Diode_SOD-123, F.Cu at (469.4, 86.9)
- added D170: Diode, ScottoKeebs_Components:Diode_SOD-123, F.Cu at (469.4, 90.5)
- added D171: Diode, ScottoKeebs_Components:Diode_SOD-123, F.Cu at (469.4, 94.0)
- added D172: Diode, ScottoKeebs_Components:Diode_SOD-123, F.Cu at (469.4, 97.5)
- added D173: Diode, ScottoKeebs_Components:Diode_SOD-123, F.Cu at (469.4, 101.1)
- added D174: Diode, ScottoKeebs_Components:Diode_SOD-123, F.Cu at (469.4, 104.7)
- added D175: Diode, ScottoKeebs_Components:Diode_SOD-123, F.Cu at (469.4, 108.2)
- added D90: Diode, ScottoKeebs_Components:Diode_SOD-123, F.Cu at (426.3, 62.0)
- added D91: Diode, ScottoKeebs_Components:Diode_SOD-123, F.Cu at (426.3, 65.6)
- added D92: Diode, ScottoKeebs_Components:Diode_SOD-123, F.Cu at (426.3, 69.2)
- added D93: Diode, ScottoKeebs_Components:Diode_SOD-123, F.Cu at (426.3, 72.7)
- added D94: Diode, ScottoKeebs_Components:Diode_SOD-123, F.Cu at (426.3, 76.2)
- added D95: Diode, ScottoKeebs_Components:Diode_SOD-123, F.Cu at (426.3, 79.8)
- added D96: Diode, ScottoKeebs_Components:Diode_SOD-123, F.Cu at (426.3, 83.3)
- added D97: Diode, ScottoKeebs_Components:Diode_SOD-123, F.Cu at (426.3, 86.9)
- added D98: Diode, ScottoKeebs_Components:Diode_SOD-123, F.Cu at (426.3, 90.5)
- added D99: Diode, ScottoKeebs_Components:Diode_SOD-123, F.Cu at (426.3, 94.0)
- added D999: Diode, ScottoKeebs_Components:Diode_SOD-123, F.Cu at (469.4, 111.8)
- added S0: Keyswitch, ScottoKeebs_Hotswap:Hotswap_MX_1.00u, F.Cu at (300.5, 68.0)
- added S1: Keyswitch, ScottoKeebs_Hotswap:Hotswap_MX_1.00u, F.Cu at (300.5, 83.6)
- added S10: Keyswitch, ScottoKeebs_Hotswap:Hotswap_MX_1.00u, F.Cu at (300.5, 223.6)
- added S11: Keyswitch, ScottoKeebs_Hotswap:Hotswap_MX_1.00u, F.Cu at (317.1, 68.0)
- added S12: Keyswitch, ScottoKeebs_Hotswap:Hotswap_MX_1.00u, F.Cu at (317.1, 83.6)
- added S13: Keyswitch, ScottoKeebs_Hotswap:Hotswap_MX_1.00u, F.Cu at (317.1, 99.2)
- added S14: Keyswitch, ScottoKeebs_Hotswap:Hotswap_MX_1.00u, F.Cu at (317.1, 114.7)
- added S15: Keyswitch, ScottoKeebs_Hotswap:Hotswap_MX_1.00u, F.Cu at (317.1, 130.2)
- added S16: Keyswitch, ScottoKeebs_Hotswap:Hotswap_MX_1.00u, F.Cu at (317.1, 145.8)
- added S17: Keyswitch, ScottoKeebs_Hotswap:Hotswap_MX_1.00u, F.Cu at (317.1, 161.3)
- added S18: Keyswitch, ScottoKeebs_Hotswap:Hotswap_MX_1.00u, F.Cu at (317.1, 176.9)
- added S19: Keyswitch, ScottoKeebs_Hotswap:Hotswap_MX_1.00u, F.Cu at (317.1, 192.4)
- added S2: Keyswitch, ScottoKeebs_Hotswap:Hotswap_MX_1.00u, F.Cu at (300.5, 99.2)
- added S20: Keyswitch, ScottoKeebs_Hotswap:Hotswap_MX_1.00u, F.Cu at (317.1, 208.0)
- added S21: Keyswitch, ScottoKeebs_Hotswap:Hotswap_MX_1.00u, F.Cu at (317.1, 223.6)
- added S22: Keyswitch, ScottoKeebs_Hotswap:Hotswap_MX_1.00u, F.Cu at (333.7, 68.0)
- added S23: Keyswitch, ScottoKeebs_Hotswap:Hotswap_MX_1.00u, F.Cu at (333.7, 83.6)
- added S24: Keyswitch, ScottoKeebs_Hotswap:Hotswap_MX_1.00u, F.Cu at (333.7, 99.2)
- added S25: Keyswitch, ScottoKeebs_Hotswap:Hotswap_MX_1.00u, F.Cu at (333.7, 114.7)
- added S26: Keyswitch, ScottoKeebs_Hotswap:Hotswap_MX_1.00u, F.Cu at (333.7, 130.2)
- added S27: Keyswitch, ScottoKeebs_Hotswap:Hotswap_MX_1.00u, F.Cu at (333.7, 145.8)
- added S28: Keyswitch, ScottoKeebs_Hotswap:Hotswap_MX_1.00u, F.Cu at (333.7, 161.3)
- added S29: Keyswitch, ScottoKeebs_Hotswap:Hotswap_MX_1.00u, F.Cu at (333.7, 176.9)
- added S3: Keyswitch, ScottoKeebs_Hotswap:Hotswap_MX_1.00u, F.Cu at (300.5, 114.7)
- added S30: Keyswitch, ScottoKeebs_Hotswap:Hotswap_MX_1.00u, F.Cu at (333.7, 192.4)
- added S31: Keyswitch, ScottoKeebs_Hotswap:Hotswap_MX_1.00u, F.Cu at (333.7, 208.0)
- added S32: Keyswitch, ScottoKeebs_Hotswap:Hotswap_MX_1.00u, F.Cu at (333.7, 223.6)
- added S33: Keyswitch, ScottoKeebs_Hotswap:Hotswap_MX_1.00u, F.Cu at (350.4, 68.0)
- added S34: Keyswitch, ScottoKeebs_Hotswap:Hotswap_MX_1.00u, F.Cu at (350.4, 83.6)
- added S35: Keyswitch, ScottoKeebs_Hotswap:Hotswap_MX_1.00u, F.Cu at (350.4, 99.2)
- added S36: Keyswitch, ScottoKeebs_Hotswap:Hotswap_MX_1.00u, F.Cu at (350.4, 114.7)
- added S37: Keyswitch, ScottoKeebs_Hotswap:Hotswap_MX_1.00u, F.Cu at (350.4, 130.2)
- added S38: Keyswitch, ScottoKeebs_Hotswap:Hotswap_MX_1.00u, F.Cu at (350.4, 145.8)
- added S39: Keyswitch, ScottoKeebs_Hotswap:Hotswap_MX_1.00u, F.Cu at (350.4, 161.3)
- added S4: Keyswitch, ScottoKeebs_Hotswap:Hotswap_MX_1.00u, F.Cu at (300.5, 130.2)
- added S40: Keyswitch, ScottoKeebs_Hotswap:Hotswap_MX_1.00u, F.Cu at (350.4, 176.9)
- added S41: Keyswitch, ScottoKeebs_Hotswap:Hotswap_MX_1.00u, F.Cu at (350.4, 192.4)
- added S42: Keyswitch, ScottoKeebs_Hotswap:Hotswap_MX_1.00u, F.Cu at (350.4, 208.0)
- added S43: Keyswitch, ScottoKeebs_Hotswap:Hotswap_MX_1.00u, F.Cu at (350.4, 223.6)
- added S44: Keyswitch, ScottoKeebs_Hotswap:Hotswap_MX_1.00u, F.Cu at (367.0, 68.0)
- added S45: Keyswitch, ScottoKeebs_Hotswap:Hotswap_MX_1.00u, F.Cu at (367.0, 83.6)
- added S46: Keyswitch, ScottoKeebs_Hotswap:Hotswap_MX_1.00u, F.Cu at (367.0, 99.2)
- added S47: Keyswitch, ScottoKeebs_Hotswap:Hotswap_MX_1.00u, F.Cu at (367.0, 114.7)
- added S48: Keyswitch, ScottoKeebs_Hotswap:Hotswap_MX_1.00u, F.Cu at (367.0, 130.2)
- added S49: Keyswitch, ScottoKeebs_Hotswap:Hotswap_MX_1.00u, F.Cu at (367.0, 145.8)
- added S5: Keyswitch, ScottoKeebs_Hotswap:Hotswap_MX_1.00u, F.Cu at (300.5, 145.8)
- added S50: Keyswitch, ScottoKeebs_Hotswap:Hotswap_MX_1.00u, F.Cu at (367.0, 161.3)
- added S51: Keyswitch, ScottoKeebs_Hotswap:Hotswap_MX_1.00u, F.Cu at (367.0, 176.9)
- added S52: Keyswitch, ScottoKeebs_Hotswap:Hotswap_MX_1.00u, F.Cu at (367.0, 192.4)
- added S53: Keyswitch, ScottoKeebs_Hotswap:Hotswap_MX_1.00u, F.Cu at (367.0, 208.0)
- added S54: Keyswitch, ScottoKeebs_Hotswap:Hotswap_MX_1.00u, F.Cu at (367.0, 223.6)
- added S55: Keyswitch, ScottoKeebs_Hotswap:Hotswap_MX_1.00u, F.Cu at (383.6, 68.0)
- added S56: Keyswitch, ScottoKeebs_Hotswap:Hotswap_MX_1.00u, F.Cu at (383.6, 83.6)
- added S57: Keyswitch, ScottoKeebs_Hotswap:Hotswap_MX_1.00u, F.Cu at (383.6, 99.2)
- added S58: Keyswitch, ScottoKeebs_Hotswap:Hotswap_MX_1.00u, F.Cu at (383.6, 114.7)
- added S59: Keyswitch, ScottoKeebs_Hotswap:Hotswap_MX_1.00u, F.Cu at (383.6, 130.2)
- added S6: Keyswitch, ScottoKeebs_Hotswap:Hotswap_MX_1.00u, F.Cu at (300.5, 161.3)
- added S60: Keyswitch, ScottoKeebs_Hotswap:Hotswap_MX_1.00u, F.Cu at (383.6, 145.8)
- added S61: Keyswitch, ScottoKeebs_Hotswap:Hotswap_MX_1.00u, F.Cu at (383.6, 161.3)
- added S62: Keyswitch, ScottoKeebs_Hotswap:Hotswap_MX_1.00u, F.Cu at (383.6, 176.9)
- added S63: Keyswitch, ScottoKeebs_Hotswap:Hotswap_MX_1.00u, F.Cu at (383.6, 192.4)
- added S64: Keyswitch, ScottoKeebs_Hotswap:Hotswap_MX_1.00u, F.Cu at (383.6, 208.0)
- added S65: Keyswitch, ScottoKeebs_Hotswap:Hotswap_MX_1.00u, F.Cu at (383.6, 223.6)
- added S66: Keyswitch, ScottoKeebs_Hotswap:Hotswap_MX_1.00u, F.Cu at (400.3, 68.0)
- added S67: Keyswitch, ScottoKeebs_Hotswap:Hotswap_MX_1.00u, F.Cu at (400.3, 83.6)
- added S68: Keyswitch, ScottoKeebs_Hotswap:Hotswap_MX_1.00u, F.Cu at (400.3, 99.2)
- added S69: Keyswitch, ScottoKeebs_Hotswap:Hotswap_MX_1.00u, F.Cu at (400.3, 114.7)
- added S7: Keyswitch, ScottoKeebs_Hotswap:Hotswap_MX_1.00u, F.Cu at (300.5, 176.9)
- added S70: Keyswitch, ScottoKeebs_Hotswap:Hotswap_MX_1.00u, F.Cu at (400.3, 130.2)
- added S71: Keyswitch, ScottoKeebs_Hotswap:Hotswap_MX_1.00u, F.Cu at (400.3, 145.8)
- added S72: Keyswitch, ScottoKeebs_Hotswap:Hotswap_MX_1.00u, F.Cu at (400.3, 161.3)
- added S73: Keyswitch, ScottoKeebs_Hotswap:Hotswap_MX_1.00u, F.Cu at (400.3, 176.9)
- added S74: Keyswitch, ScottoKeebs_Hotswap:Hotswap_MX_1.00u, F.Cu at (400.3, 192.4)
- added S75: Keyswitch, ScottoKeebs_Hotswap:Hotswap_MX_1.00u, F.Cu at (400.3, 208.0)
- added S76: Keyswitch, ScottoKeebs_Hotswap:Hotswap_MX_1.00u, F.Cu at (400.3, 223.6)
- added S77: Keyswitch, ScottoKeebs_Hotswap:Hotswap_MX_1.00u, F.Cu at (416.9, 68.0)
- added S78: Keyswitch, ScottoKeebs_Hotswap:Hotswap_MX_1.00u, F.Cu at (416.9, 83.6)
- added S79: Keyswitch, ScottoKeebs_Hotswap:Hotswap_MX_1.00u, F.Cu at (416.9, 99.2)
- added S8: Keyswitch, ScottoKeebs_Hotswap:Hotswap_MX_1.00u, F.Cu at (300.5, 192.4)
- added S80: Keyswitch, ScottoKeebs_Hotswap:Hotswap_MX_1.00u, F.Cu at (416.9, 114.7)
- added S81: Keyswitch, ScottoKeebs_Hotswap:Hotswap_MX_1.00u, F.Cu at (416.9, 130.2)
- added S82: Keyswitch, ScottoKeebs_Hotswap:Hotswap_MX_1.00u, F.Cu at (416.9, 145.8)
- added S83: Keyswitch, ScottoKeebs_Hotswap:Hotswap_MX_1.00u, F.Cu at (416.9, 161.3)
- added S84: Keyswitch, ScottoKeebs_Hotswap:Hotswap_MX_1.00u, F.Cu at (416.9, 176.9)
- added S85: Keyswitch, ScottoKeebs_Hotswap:Hotswap_MX_1.00u, F.Cu at (416.9, 192.4)
- added S86: Keyswitch, ScottoKeebs_Hotswap:Hotswap_MX_1.00u, F.Cu at (416.9, 208.0)
- added S9: Keyswitch, ScottoKeebs_Hotswap:Hotswap_MX_1.00u, F.Cu at (300.5, 208.0)
- moved H1 335.7 mm to (171.0, 245.0)
- moved H2 335.7 mm to (185.0, 245.0)
- moved H3 335.7 mm to (171.0, 257.0)
- moved H4 335.7 mm to (185.0, 257.0)
