File: v2/Matrix/v2.kicad_sch (KiCad schematic)
At the start: 360 parts, among them J2 Conn_01x16, K0 ESC, K1 F1, K10 F10, K11 F11, K12 F12, K13 <i class='kb kb-Unicode-Print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, K14 INS, K15 DEL, K16 |,\, K17 !,,,,,,,,,1, K18 ",@,,,,,,,,2, K19 #,£,,,,,,,,3, K2 F2, K20 $,§,,,,,,,,4, K21 %,€,,,,,,,,5, K22 &,,,,,,,,,6, K23 /,{,,,,,,,,7, K24 (,[,,,,,,,,8, K25 ),],,,,,,,,9, K26 =,},,,,,,,,0, K27 ?,', K28 »,«, K29 BACKSPACE, K3 F3, K30 Blank, K31 PGUP, K32 TAB, K33 Q, K34 W, K35 E, K36 R, K37 T, K38 Y, K39 U, K4 F4, K40 I, K41 O, K42 P, K43 *,+, K44 `,´, K45 |,\, K46 PGDN, K47 CAPS, K48 A, K49 S, K5 F5, K50 D, K51 F, K52 G, K53 H, K54 J, K55 K, K56 L, K57 Ç, K58 ª,º, K59 ^,~~, K6 F6, K60 ENTER, K61 HOME, K62 SHIFT, K63 Z, K64 X, K65 C, K66 V, K67 B, K68 N, K69 M, K7 F7, K70 ;,,, K71 :,., K72 -,_, K73 >,,,,,,,,,<, K74 SHIFT, K75 END, K76 ∧, K77 Blank, K78 CTRL, K79 SUPER, K8 F8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

Commit message: Updated the kicad schematics.
Parts:
- D100, D101, D102, D103, D104, D105, D106, D107, D108, D109, D110, D111, D112, D113, D114, D115, D116, D117, D118, D119, D120, D121, D122, D123, D124, D125, D126, D127, D128, D129, D130, D131, D132, D133, D134, D135, D136, D137, D138, D139, D140, D141, D142, D143, D144, D145, D146, D147, D148, D149, D150, D151, D152, D153, D154, D155, D156, D157, D158, D159, D160, D161, D162, D163, D164, D165, D166, D167, D168, D169, D170, D171, D172, D173, D174, D175, D90, D91, D92, D93, D94, D95, D96, D97, D98, D99, D999: footprint (none) -> ScottoKeebs_Components:Diode_SOD-123
- S0, S1, S10, S11, S12, S13, S14, S15, S16, S17, S18, S19, S2, S20, S21, S22, S23, S24, S25, S26, S27, S28, S29, S3, S30, S31, S32, S33, S34, S35, S36, S37, S38, S39, S4, S40, S41, S42, S43, S44, S45, S46, S47, S48, S49, S5, S50, S51, S52, S53, S54, S55, S56, S57, S58, S59, S6, S60, S61, S62, S63, S64, S65, S66, S67, S68, S69, S7, S70, S71, S72, S73, S74, S75, S76, S77, S78, S79, S8, S80, S81, S82, S83, S84, S85, S86, S9: footprint (none) -> ScottoKeebs_Hotswap:Hotswap_MX_1.00u
