File: v1/Matrix/v1.kicad_pcb (KiCad board)
At the start: 2 copper layers, 180 parts, among them J1 Conn_01x06, J2 Conn_01x16

Commit message: additions to the v1 pcb and schematics
Parts:
- removed D100, D101, D102, D103, D104, D105, D106, D107, D108, D109, D110, D111, D112, D113, D114, D115, D116, D117, D118, D119, D120, D121, D122, D123, D124, D125, D126, D127, D128, D129, D130, D131, D132, D133, D134, D135, D136, D137, D138, D139, D140, D141, D142, D143, D144, D145, D146, D147, D148, D149, D150, D151, D152, D153, D154, D155, D156, D157, D158, D159, D160, D161, D162, D163, D164, D165, D166, D167, D168, D169, D170, D171, D172, D173, D174, D175, D90, D91, D92, D93, D94, D95, D96, D97, D98, D99, D999: Diode, ScottoKeebs_Components:Diode_SOD-123
- added D0: Diode, ScottoKeebs_Components:Diode_DO-35, F.Cu at (149.1, 164.4)
- added D1: Diode, ScottoKeebs_Components:Diode_DO-35, F.Cu at (149.1, 167.9)
- added D10: Diode, ScottoKeebs_Components:Diode_DO-35, F.Cu at (149.1, 199.9)
- added D11: Diode, ScottoKeebs_Components:Diode_DO-35, F.Cu at (149.1, 203.4)
- added D12: Diode, ScottoKeebs_Components:Diode_DO-35, F.Cu at (149.1, 207.0)
- added D13: Diode, ScottoKeebs_Components:Diode_DO-35, F.Cu at (149.1, 210.5)
- added D14: Diode, ScottoKeebs_Components:Diode_DO-35, F.Cu at (149.1, 214.1)
- added D15: Diode, ScottoKeebs_Components:Diode_DO-35, F.Cu at (149.1, 217.6)
- added D16: Diode, ScottoKeebs_Components:Diode_DO-35, F.Cu at (149.1, 221.2)
- added D17: Diode, ScottoKeebs_Components:Diode_DO-35, F.Cu at (149.1, 224.7)
- added D18: Diode, ScottoKeebs_Components:Diode_DO-35, F.Cu at (159.9, 164.4)
- added D19: Diode, ScottoKeebs_Components:Diode_DO-35, F.Cu at (159.9, 167.9)
- added D2: Diode, ScottoKeebs_Components:Diode_DO-35, F.Cu at (149.1, 171.5)
- added D20: Diode, ScottoKeebs_Components:Diode_DO-35, F.Cu at (159.9, 171.5)
- added D21: Diode, ScottoKeebs_Components:Diode_DO-35, F.Cu at (159.9, 175.0)
- added D22: Diode, ScottoKeebs_Components:Diode_DO-35, F.Cu at (159.9, 178.6)
- added D23: Diode, ScottoKeebs_Components:Diode_DO-35, F.Cu at (159.9, 182.1)
- added D24: Diode, ScottoKeebs_Components:Diode_DO-35, F.Cu at (159.9, 185.7)
- added D25: Diode, ScottoKeebs_Components:Diode_DO-35, F.Cu at (159.9, 189.2)
- added D26: Diode, ScottoKeebs_Components:Diode_DO-35, F.Cu at (159.9, 192.8)
- added D27: Diode, ScottoKeebs_Components:Diode_DO-35, F.Cu at (159.9, 196.3)
- added D28: Diode, ScottoKeebs_Components:Diode_DO-35, F.Cu at (159.9, 199.9)
- added D29: Diode, ScottoKeebs_Components:Diode_DO-35, F.Cu at (159.9, 203.4)
- added D3: Diode, ScottoKeebs_Components:Diode_DO-35, F.Cu at (149.1, 175.0)
- added D30: Diode, ScottoKeebs_Components:Diode_DO-35, F.Cu at (159.9, 207.0)
- added D31: Diode, ScottoKeebs_Components:Diode_DO-35, F.Cu at (159.9, 210.5)
- added D32: Diode, ScottoKeebs_Components:Diode_DO-35, F.Cu at (159.9, 214.1)
- added D33: Diode, ScottoKeebs_Components:Diode_DO-35, F.Cu at (159.9, 217.6)
- added D34: Diode, ScottoKeebs_Components:Diode_DO-35, F.Cu at (159.9, 221.2)
- added D35: Diode, ScottoKeebs_Components:Diode_DO-35, F.Cu at (159.9, 224.7)
- added D36: Diode, ScottoKeebs_Components:Diode_DO-35, F.Cu at (170.6, 164.4)
- added D37: Diode, ScottoKeebs_Components:Diode_DO-35, F.Cu at (170.6, 167.9)
- added D38: Diode, ScottoKeebs_Components:Diode_DO-35, F.Cu at (170.6, 171.5)
- added D39: Diode, ScottoKeebs_Components:Diode_DO-35, F.Cu at (170.6, 175.0)
- added D4: Diode, ScottoKeebs_Components:Diode_DO-35, F.Cu at (149.1, 178.6)
- added D40: Diode, ScottoKeebs_Components:Diode_DO-35, F.Cu at (170.6, 178.6)
- added D41: Diode, ScottoKeebs_Components:Diode_DO-35, F.Cu at (170.6, 182.1)
- added D42: Diode, ScottoKeebs_Components:Diode_DO-35, F.Cu at (170.6, 185.7)
- added D43: Diode, ScottoKeebs_Components:Diode_DO-35, F.Cu at (170.6, 189.2)
- added D44: Diode, ScottoKeebs_Components:Diode_DO-35, F.Cu at (170.6, 192.8)
- added D45: Diode, ScottoKeebs_Components:Diode_DO-35, F.Cu at (170.6, 196.3)
- added D46: Diode, ScottoKeebs_Components:Diode_DO-35, F.Cu at (170.6, 199.9)
- added D47: Diode, ScottoKeebs_Components:Diode_DO-35, F.Cu at (170.6, 203.4)
- added D48: Diode, ScottoKeebs_Components:Diode_DO-35, F.Cu at (170.6, 207.0)
- added D49: Diode, ScottoKeebs_Components:Diode_DO-35, F.Cu at (170.6, 210.5)
- added D5: Diode, ScottoKeebs_Components:Diode_DO-35, F.Cu at (149.1, 182.1)
- added D50: Diode, ScottoKeebs_Components:Diode_DO-35, F.Cu at (170.6, 214.1)
- added D51: Diode, ScottoKeebs_Components:Diode_DO-35, F.Cu at (170.6, 217.6)
- added D52: Diode, ScottoKeebs_Components:Diode_DO-35, F.Cu at (170.6, 221.2)
- added D53: Diode, ScottoKeebs_Components:Diode_DO-35, F.Cu at (170.6, 224.7)
- added D54: Diode, ScottoKeebs_Components:Diode_DO-35, F.Cu at (181.4, 164.4)
- added D55: Diode, ScottoKeebs_Components:Diode_DO-35, F.Cu at (181.4, 167.9)
- added D56: Diode, ScottoKeebs_Components:Diode_DO-35, F.Cu at (181.4, 171.5)
- added D57: Diode, ScottoKeebs_Components:Diode_DO-35, F.Cu at (181.4, 175.0)
- added D58: Diode, ScottoKeebs_Components:Diode_DO-35, F.Cu at (181.4, 178.6)
- added D59: Diode, ScottoKeebs_Components:Diode_DO-35, F.Cu at (181.4, 182.1)
- added D6: Diode, ScottoKeebs_Components:Diode_DO-35, F.Cu at (149.1, 185.7)
- added D60: Diode, ScottoKeebs_Components:Diode_DO-35, F.Cu at (181.4, 185.7)
- added D61: Diode, ScottoKeebs_Components:Diode_DO-35, F.Cu at (181.4, 189.2)
- added D62: Diode, ScottoKeebs_Components:Diode_DO-35, F.Cu at (181.4, 192.8)
- added D63: Diode, ScottoKeebs_Components:Diode_DO-35, F.Cu at (181.4, 196.3)
- added D64: Diode, ScottoKeebs_Components:Diode_DO-35, F.Cu at (181.4, 199.9)
- added D65: Diode, ScottoKeebs_Components:Diode_DO-35, F.Cu at (181.4, 203.4)
- added D66: Diode, ScottoKeebs_Components:Diode_DO-35, F.Cu at (181.4, 207.0)
- added D67: Diode, ScottoKeebs_Components:Diode_DO-35, F.Cu at (181.4, 210.5)
- added D68: Diode, ScottoKeebs_Components:Diode_DO-35, F.Cu at (181.4, 214.1)
- added D69: Diode, ScottoKeebs_Components:Diode_DO-35, F.Cu at (181.4, 217.6)
- added D7: Diode, ScottoKeebs_Components:Diode_DO-35, F.Cu at (149.1, 189.2)
- added D70: Diode, ScottoKeebs_Components:Diode_DO-35, F.Cu at (181.4, 221.2)
- added D71: Diode, ScottoKeebs_Components:Diode_DO-35, F.Cu at (181.4, 224.7)
- added D72: Diode, ScottoKeebs_Components:Diode_DO-35, F.Cu at (192.2, 164.4)
- added D73: Diode, ScottoKeebs_Components:Diode_DO-35, F.Cu at (192.2, 167.9)
- added D74: Diode, ScottoKeebs_Components:Diode_DO-35, F.Cu at (192.2, 171.5)
- added D75: Diode, ScottoKeebs_Components:Diode_DO-35, F.Cu at (192.2, 175.0)
- added D76: Diode, ScottoKeebs_Components:Diode_DO-35, F.Cu at (192.2, 178.6)
- added D77: Diode, ScottoKeebs_Components:Diode_DO-35, F.Cu at (192.2, 182.1)
- added D78: Diode, ScottoKeebs_Components:Diode_DO-35, F.Cu at (192.2, 185.7)
- added D79: Diode, ScottoKeebs_Components:Diode_DO-35, F.Cu at (192.2, 189.2)
- added D8: Diode, ScottoKeebs_Components:Diode_DO-35, F.Cu at (149.1, 192.8)
- added D80: Diode, ScottoKeebs_Components:Diode_DO-35, F.Cu at (192.2, 192.8)
- added D81: Diode, ScottoKeebs_Components:Diode_DO-35, F.Cu at (192.2, 196.3)
- added D82: Diode, ScottoKeebs_Components:Diode_DO-35, F.Cu at (192.2, 199.9)
- added D83: Diode, ScottoKeebs_Components:Diode_DO-35, F.Cu at (192.2, 203.4)
- added D84: Diode, ScottoKeebs_Components:Diode_DO-35, F.Cu at (192.2, 207.0)
- added D85: Diode, ScottoKeebs_Components:Diode_DO-35, F.Cu at (192.2, 210.5)
- added D86: Diode, ScottoKeebs_Components:Diode_DO-35, F.Cu at (192.2, 214.1)
- added D9: Diode, ScottoKeebs_Components:Diode_DO-35, F.Cu at (149.1, 196.3)
- moved H1 335.1 mm to (25.9, 26.0)
- moved S30 286.8 mm to (349.8, 66.4)
- moved S15 283.5 mm to (349.8, 42.6)
- moved S10 269.2 mm to (245.0, 42.6)
- moved H3 261.2 mm to (30.7, 161.7)
- moved S14 255.5 mm to (326.0, 42.6)
- moved H2 245.3 mm to (366.5, 26.0)
- moved S9 245.1 mm to (226.0, 42.6)
- moved S29 244.4 mm to (309.3, 66.4)
- moved S13 232.0 mm to (306.9, 42.6)
- moved S43 229.3 mm to (283.1, 85.5)
- moved S8 221.1 mm to (206.9, 42.6)
- moved S28 214.0 mm to (283.1, 66.4)
- moved S45 211.0 mm to (349.8, 85.5)
- moved S75 208.1 mm to (349.5, 123.6)
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Connections:
- S47 pad 1: /Col0 -> /Col1
- S48 pad 1: /Col1 -> /Col2
- S49 pad 1: /Col1 -> /Col3
- S50 pad 1: /Col2 -> /Col4
- S51 pad 1: /Col2 -> /Col5
- S52 pad 1: /Col3 -> /Col6
- S53 pad 1: /Col3 -> /Col7
- S54 pad 1: /Col4 -> /Col8
- S55 pad 1: /Col4 -> /Col9
- S56 pad 1: /Col5 -> /Col10
- S57 pad 1: /Col5 -> /Col11
- S58 pad 1: /Col6 -> /Col12
- S59 pad 1: /Col6 -> /Col13
- S60 pad 1: /Col7 -> /Col14
- S61 pad 1: /Col7 -> /Col0
- S62 pad 1: /Col8 -> /Col1
- S63 pad 1: /Col8 -> /Col2
- S64 pad 1: /Col9 -> /Col3
- S65 pad 1: /Col9 -> /Col4
- S66 pad 1: /Col10 -> /Col5
- S67 pad 1: /Col10 -> /Col6
- S68 pad 1: /Col11 -> /Col7
- S69 pad 1: /Col11 -> /Col8
- S70 pad 1: /Col12 -> /Col9
- S71 pad 1: /Col12 -> /Col10
- S72 pad 1: /Col13 -> /Col11
- S73 pad 1: /Col13 -> /Col12
- S74 pad 1: /Col14 -> /Col13
Routing:
- net /Col2: track 0.00 -> 243.8 mm
- net /Col3: track 0.00 -> 220.8 mm
- net /Col8: track 0.00 -> 196.3 mm
- net /Col1: track 0.00 -> 190.0 mm
- net /Col6: track 0.00 -> 188.3 mm
- net /Col7: track 0.00 -> 186.9 mm
- net /Col5: track 0.00 -> 185.5 mm
- net /Col4: track 0.00 -> 140.5 mm
- net /Col0: track 0.00 -> 111.2 mm
- net /Col13: track 0.00 -> 93.5 mm
- net /Col14: track 0.00 -> 92.3 mm
- net /Col12: track 0.00 -> 84.9 mm
- net /Col10: track 0.00 -> 81.0 mm
- net /Col9: track 0.00 -> 81.0 mm
- net /Col11: track 0.00 -> 81.0 mm
