File: Modules/NumpadMatrix/v2/Keyboard NumPad v1.kicad_sch (KiCad schematic)
At the start: 55 parts, among them U2 ESP32-C3_SUPERMINI_SMD

Commit message: Update of Module V2  x_x
Connections:
- net Coluna 0: no longer S27.1
- net Coluna 3: no longer S25.1, S26.1
- net Linha 4: now also D27.1 (K)
- net Linha 5: no longer D27.1 (K)
- net Coluna 4: now reaches U2.10 (GPIO10)
- net Coluna 4: now also S25.1, S26.1, S27.1
Other:
- moved on the sheet: D25, D26, D27, S25, S26, S27
