File: Modules/NumpadMatrix/v2/Keyboard NumPad v1.kicad_pcb (KiCad board)
At the start: 2 copper layers, 80.2 x 123 mm, 60 parts, among them U2 ESP32-C3_SUPERMINI_SMD

Commit message: message here
Other:
- board size 80.2 x 123 mm -> 80.3 x 123.2 mm
Changed lines of the file:
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@@
 	)
 	(gr_arc
-		(start 26.81 149.93)
-		(mid 25.395786 149.344214)
-		(end 24.81 147.93)
+		(start 24.747001 29.049)
+		(mid 25.3617 27.618465)
+		(end 26.798958 27.019652)
 		(stroke
 			(width 0.05)
@@
 	(gr_line
 		(start 24.81 122.18)
-		(end 24.81 147.93)
-		(stroke
-			(width 0.05)
-			(type default)
-		)
-		(layer "Edge.Cuts")
-	)
-	(gr_arc
-		(start 105.06 147.93)
-		(mid 104.474214 149.344214)
-		(end 103.06 149.93)
+		(end 24.736 148.19)
 		(stroke
 			(width 0.05)
@@
 	)
 	(gr_line
-		(start 83.81 149.93)
-		(end 26.81 149.93)
+		(start 26.799 27.024)
+		(end 103.005 27.058)
 		(stroke
 			(width 0.05)
@@
 		(layer "Edge.Cuts")
 	)
-	(gr_line
-		(start 36.81 26.93)
-		(end 26.81 26.93)
+	(gr_arc
+		(start 26.812982 150.243207)
+		(mid 25.354448 149.641511)
+		(end 24.736 148.19)
 		(stroke
 			(width 0.05)
@@
 		(layer "Edge.Cuts")
 	)
-	(gr_line
-		(start 36.81 26.93)
-		(end 103.06 26.93)
+	(gr_arc
+		(start 103.005 27.058)
+		(mid 104.456621 27.653332)
+		(end 105.070837 29.097065)
 		(stroke
 			(width 0.05)
@@
 	)
 	(gr_line
-		(start 83.81 149.93)
-		(end 103.06 149.93)
+		(start 26.813 150.237)
+		(end 102.996 150.235)
 		(stroke
 			(width 0.05)
@@
 	)
 	(gr_arc
-		(start 24.81 28.93)
-		(mid 25.395786 27.515786)
-		(end 26.81 26.93)
-		(stroke
-			(width 0.05)
-			(type default)
-		)
-		(layer "Edge.Cuts")
-	)
-	(gr_arc
-		(start 103.06 26.93)
-		(mid 104.474214 27.515786)
-		(end 105.06 28.93)
-		(stroke
-			(width 0.05)
-			(type default)
-		)
-		(layer "Edge.Cuts")
-	)
-	(gr_line
-		(start 24.81 116.93)
-		(end 24.81 28.93)
+		(start 105.075152 148.181)
+		(mid 104.464639 149.642317)
+		(end 102.996 150.235)
 		(stroke
 			(width 0.05)
@@
 	)
 	(gr_line
-		(start 105.06 112.18)
-		(end 105.06 147.93)
+		(start 24.742 116.94)
+		(end 24.747 29.049)
 		(stroke
 			(width 0.05)
@@
 	)
 	(gr_line
-		(start 105.06 112.18)
-		(end 105.06 28.93)
+		(start 105.074 148.181)
+		(end 105.076 29.097)
 		(stroke
 			(width 0.05)
@@
 		(polygon
 			(pts
-				(xy 14.90375 17.21125) (xy 117.2975 19.5925) (xy 114.91625 150.56125) (xy 14.90375 160.08625)
+				(xy 26.81 25.93) (xy 23.81 28.93) (xy 23.81 148.93) (xy 26.81 150.93) (xy 103.81 150.93) (xy 105.81 148.93)
+				(xy 105.81 27.93) (xy 103.81 25.93)
 			)
 		)
