File: ControllerBoard/v0/keyboard ControlBoard v0.kicad_pcb (KiCad board)
At the start: 2 copper layers, 1 part, among them U1 ESP32-S3-DEVKITC-1-N8R2

Commit message: ControlBoard V0 :P
Parts:
- added SW1: RotaryEncoder_Switch, ToxyzRotaryEncoder-Switch:RotaryEncoder_Toxyz_Switch_Horizontal, F.Cu at (110.2, 68.2)
- U1: footprint ESP32-S3:XCVR_ESP32-S3-DEVKITC-1-N8R2 -> Esp32-S3-DevKit:XCVR_ESP32-S3-DEVKITC-1-N8R2
- moved U1 52.2 mm to (82.6, 90.6)
Connections:
- U1 pad J1_1: unconnected-(U1-3V3-PadJ1_1) -> LED
- U1 pad J1_10: unconnected-(U1-GPIO17-PadJ1_10) -> LCD_CS
- U1 pad J1_22: unconnected-(U1-GND-PadJ1_22) -> GND
- U1 pad J1_4: unconnected-(U1-GPIO4-PadJ1_4) -> SDO (MISO)
- U1 pad J1_6: unconnected-(U1-GPIO6-PadJ1_6) -> SCK
- U1 pad J1_7: unconnected-(U1-GPIO7-PadJ1_7) -> SDI (MOSI)
- U1 pad J1_8: unconnected-(U1-GPIO15-PadJ1_8) -> LCD_RS
- U1 pad J1_9: unconnected-(U1-GPIO16-PadJ1_9) -> LCD_RST
- U1 pad J3_11: unconnected-(U1-GPIO37-PadJ3_11) -> S1 Switch
- U1 pad J3_12: unconnected-(U1-GPIO36-PadJ3_12) -> RotaryEncoder B
- U1 pad J3_13: unconnected-(U1-GPIO35-PadJ3_13) -> RotaryEncoder A
