File: ControllerBoard/v0/ControlBoard v0.kicad_pcb (KiCad board)
At the start: 2 copper layers, 2 parts, among them SW1 RotaryEncoder_Switch, U1 ESP32-S3-DEVKITC-1-N8R2

Commit message: resolvendo merda :-:
Parts:
- removed SW1: RotaryEncoder_Switch, ToxyzRotaryEncoder-Switch:RotaryEncoder_Toxyz_Switch_Horizontal
- U1: footprint Esp32-S3-DevKit:XCVR_ESP32-S3-DEVKITC-1-N8R2 -> ESP32-S3:XCVR_ESP32-S3-DEVKITC-1-N8R2
- moved U1 52.2 mm to (38.2, 63.1)
Connections:
- U1 pad J1_1: LED -> unconnected-(U1-3V3-PadJ1_1)
- U1 pad J1_10: LCD_CS -> unconnected-(U1-GPIO17-PadJ1_10)
- U1 pad J1_22: GND -> unconnected-(U1-GND-PadJ1_22)
- U1 pad J1_4: SDO (MISO) -> unconnected-(U1-GPIO4-PadJ1_4)
- U1 pad J1_6: SCK -> unconnected-(U1-GPIO6-PadJ1_6)
- U1 pad J1_7: SDI (MOSI) -> unconnected-(U1-GPIO7-PadJ1_7)
- U1 pad J1_8: LCD_RS -> unconnected-(U1-GPIO15-PadJ1_8)
- U1 pad J1_9: LCD_RST -> unconnected-(U1-GPIO16-PadJ1_9)
- U1 pad J3_11: S1 Switch -> unconnected-(U1-GPIO37-PadJ3_11)
- U1 pad J3_12: RotaryEncoder B -> unconnected-(U1-GPIO36-PadJ3_12)
- U1 pad J3_13: RotaryEncoder A -> unconnected-(U1-GPIO35-PadJ3_13)
